File: CAN_DISPLAY/PowerSuply.kicad_sch (KiCad schematic)
At the start: 29 parts, among them J10 DCDC 5V 3A, J15 CHARGER, J6 12V, J8 DCDC 5V, U4 AMS1117-3.3

Commit message: Add SW
Parts:
- removed J15: CHARGER, TerminalBlock:TerminalBlock_bornier-4_P5.08mm, symbol Connector:Screw_Terminal_01x04
- added J5: Power, TerminalBlock:TerminalBlock_bornier-5_P5.08mm, symbol Connector:Screw_Terminal_01x05
- added JP19: Open, Jumper:SolderJumper-2_P1.3mm_Open_RoundedPad1.0x1.5mm, symbol Jumper:SolderJumper_2_Open
- D3, D4: footprint LED_SMD:LED_1210_3225Metric -> LED_SMD:LED_0805_2012Metric_Pad1.15x1.40mm_HandSolder
Connections:
- net +12V: now also J5.5 (Pin_5), JP19.1 (A); no longer JP19.1 (A)
- net 12V_FL: now also J5.2 (Pin_2)
- net GND: now also J5.1 (Pin_1), J5.3 (Pin_3)
- new net: J5.4 (Pin_4), JP19.1 (A), JP19.2 (B)
Other:
- moved on the sheet: JP19
Changed lines of the file:
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@@
   (junction (at 163.83 124.46) (diameter 0) (color 0 0 0 0)
   )
+  (junction (at 45.72 77.47) (diameter 0) (color 0 0 0 0)
+  )
   (junction (at 148.59 175.26) (diameter 0) (color 0 0 0 0)
   )
@@
   (junction (at 34.29 85.09) (diameter 0) (color 0 0 0 0)
   )
-  (junction (at 38.1 77.47) (diameter 0) (color 0 0 0 0)
+  (junction (at 34.29 74.93) (diameter 0) (color 0 0 0 0)
   )
   (junction (at 209.55 133.35) (diameter 0) (color 0 0 0 0)
@@
     (stroke (width 0) (type default))
   )
+  (wire (pts (xy 45.72 77.47) (xy 46.99 77.47))
+    (stroke (width 0) (type default))
+  )
   (wire (pts (xy 139.7 113.03) (xy 148.59 113.03))
     (stroke (width 0) (type default))
@@
     (stroke (width 0) (type default))
   )
+  (wire (pts (xy 31.75 74.93) (xy 34.29 74.93))
+    (stroke (width 0) (type default))
+  )
   (wire (pts (xy 80.01 43.18) (xy 90.17 43.18))
     (stroke (width 0) (type default))
@@
     (stroke (width 0) (type default))
   )
-  (wire (pts (xy 31.75 82.55) (xy 50.8 82.55))
-    (stroke (width 0) (type default))
-  )
   (wire (pts (xy 107.95 43.18) (xy 107.95 45.72))
     (stroke (width 0) (type default))
@@
     (stroke (width 0) (type default))
   )
+  (wire (pts (xy 31.75 82.55) (xy 55.88 82.55))
+    (stroke (width 0) (type default))
+  )
   (wire (pts (xy 255.27 33.02) (xy 255.27 36.83))
     (stroke (width 0) (type default))
@@
     (stroke (width 0) (type default))
   )
-  (wire (pts (xy 38.1 77.47) (xy 38.1 74.93))
+  (wire (pts (xy 34.29 74.93) (xy 34.29 72.39))
     (stroke (width 0) (type default))
   )
@@
     (stroke (width 0) (type default))
   )
+  (wire (pts (xy 45.72 74.93) (xy 45.72 77.47))
+    (stroke (width 0) (type default))
+  )
   (wire (pts (xy 90.17 48.26) (xy 90.17 50.8))
     (stroke (width 0) (type default))
@@
     (stroke (width 0) (type default))
   )
+  (wire (pts (xy 41.91 74.93) (xy 45.72 74.93))
+    (stroke (width 0) (type default))
+  )
   (wire (pts (xy 148.59 175.26) (xy 148.59 173.99))
     (stroke (width 0) (type default))
   )
-  (wire (pts (xy 38.1 77.47) (xy 40.64 77.47))
+  (wire (pts (xy 31.75 77.47) (xy 45.72 77.47))
     (stroke (width 0) (type default))
   )
@@
     (stroke (width 0) (type default))
   )
-  (wire (pts (xy 31.75 77.47) (xy 38.1 77.47))
-    (stroke (width 0) (type default))
-  )
   (wire (pts (xy 262.89 66.675) (xy 262.89 67.945))
     (stroke (width 0) (type default))
@@
     (stroke (width 0) (type default))
   )
-  (wire (pts (xy 50.8 82.55) (xy 50.8 77.47))
+  (wire (pts (xy 55.88 82.55) (xy 55.88 77.47))
     (stroke (width 0) (type default))
   )
@@
     (stroke (width 0) (type default))
   )
-  (wire (pts (xy 50.8 77.47) (xy 48.26 77.47))
+  (wire (pts (xy 55.88 77.47) (xy 54.61 77.47))
     (stroke (width 0) (type default))
   )
@@
     (effects (font (size 1.27 1.27)) (justify right bottom))
   )
-  (label "12V_FL" (at 44.45 82.55 180) (fields_autoplaced)
+  (label "12V_FL" (at 49.53 82.55 180) (fields_autoplaced)
     (effects (font (size 1.27 1.27)) (justify right bottom))
   )
@@
       (effects (font (size 1.27 1.27)) (justify right))
     )
-    (property "Footprint" "LED_SMD:LED_1210_3225Metric" (at 262.89 64.135 90)
+    (property "Footprint" "LED_SMD:LED_0805_2012Metric_Pad1.15x1.40mm_HandSolder" (at 262.89 64.135 90)
       (effects (font (size 1.27 1.27)) hide)
     )
@@
     )
   )
+  (symbol (lib_id "Connector:Screw_Terminal_01x05") (at 26.67 80.01 180) (unit 1)
+    (in_bom yes) (on_board yes) (dnp no) (fields_autoplaced)
+    (property "Reference" "J5" (at 26.67 68.58 0)
+      (effects (font (size 1.27 1.27)))
+    )
+    (property "Value" "Power" (at 26.67 71.12 0)
+      (effects (font (size 1.27 1.27)))
+    )
+    (property "Footprint" "TerminalBlock:TerminalBlock_bornier-5_P5.08mm" (at 26.67 80.01 0)
+      (effects (font (size 1.27 1.27)) hide)
+    )
+    (property "Datasheet" "~" (at 26.67 80.01 0)
+      (effects (font (size 1.27 1.27)) hide)
+    )
+    (pin "1")
+    (pin "2")
+    (pin "3")
+    (pin "4")
+    (pin "5")
+    (instances
+      (project "CAN_DISPLAY"
+        (path "/7b7bcc60-3b35-483b-8f75-db7ec854d7bb/64058649-9106-47b8-8357-4a2d690c60fd"
+          (reference "J5") (unit 1)
+        )
+      )
+    )
+  )
   (symbol (lib_id "Device:C_Small") (at 214.63 128.27 0) (unit 1)
     (in_bom yes) (on_board yes) (dnp no)
@@
       (effects (font (size 1.27 1.27)) (justify right))
     )
-    (property "Footprint" "LED_SMD:LED_1210_3225Metric" (at 107.95 53.34 90)
+    (property "Footprint" "LED_SMD:LED_0805_2012Metric_Pad1.15x1.40mm_HandSolder" (at 107.95 53.34 90)
       (effects (font (size 1.27 1.27)) hide)
     )
@@
     )
   )
-  (symbol (lib_id "Jumper:SolderJumper_2_Open") (at 44.45 77.47 0) (unit 1)
-    (in_bom yes) (on_board yes) (dnp no)
-    (property "Reference" "JP19" (at 46.99 71.755 90)
+  (symbol (lib_id "Jumper:SolderJumper_2_Open") (at 50.8 77.47 0) (unit 1)
+    (in_bom yes) (on_board yes) (dnp no)
+    (property "Reference" "JP19" (at 53.34 71.755 90)
       (effects (font (size 1.27 1.27)) (justify right))
     )
-    (property "Value" "Open" (at 42.545 71.755 90)
+    (property "Value" "Open" (at 48.895 71.755 90)
       (effects (font (size 1.27 1.27)) (justify right))
     )
-    (property "Footprint" "Jumper:SolderJumper-2_P1.3mm_Open_RoundedPad1.0x1.5mm" (at 44.45 77.47 0)
-      (effects (font (size 1.27 1.27)) hide)
-    )
-    (property "Datasheet" "~" (at 44.45 77.47 0)
+    (property "Footprint" "Jumper:SolderJumper-2_P1.3mm_Open_RoundedPad1.0x1.5mm" (at 50.8 77.47 0)
+      (effects (font (size 1.27 1.27)) hide)
+    )
+    (property "Datasheet" "~" (at 50.8 77.47 0)
       (effects (font (size 1.27 1.27)) hide)
     )
@@
     )
   )
-  (symbol (lib_id "power:+12V") (at 38.1 74.93 0) (unit 1)
-    (in_bom yes) (on_board yes) (dnp no) (fields_autoplaced)
-    (property "Reference" "#PWR090" (at 38.1 78.74 0)
-      (effects (font (size 1.27 1.27)) hide)
-    )
-    (property "Value" "+12V" (at 38.1 69.85 0)
-      (effects (font (size 1.27 1.27)))
-    )
-    (property "Footprint" "" (at 38.1 74.93 0)
-      (effects (font (size 1.27 1.27)) hide)
-    )
-    (property "Datasheet" "" (at 38.1 74.93 0)
+  (symbol (lib_id "power:+12V") (at 34.29 72.39 0) (unit 1)
+    (in_bom yes) (on_board yes) (dnp no) (fields_autoplaced)
+    (property "Reference" "#PWR090" (at 34.29 76.2 0)
+      (effects (font (size 1.27 1.27)) hide)
+    )
+    (property "Value" "+12V" (at 34.29 67.31 0)
+      (effects (font (size 1.27 1.27)))
+    )
+    (property "Footprint" "" (at 34.29 72.39 0)
+      (effects (font (size 1.27 1.27)) hide)
+    )
+    (property "Datasheet" "" (at 34.29 72.39 0)
       (effects (font (size 1.27 1.27)) hide)
     )
@@
     )
   )
+  (symbol (lib_id "Jumper:SolderJumper_2_Open") (at 38.1 74.93 0) (unit 1)
+    (in_bom yes) (on_board yes) (dnp no)
+    (property "Reference" "JP19" (at 40.64 69.215 90)
+      (effects (font (size 1.27 1.27)) (justify right))
+    )
+    (property "Value" "Open" (at 36.195 69.215 90)
+      (effects (font (size 1.27 1.27)) (justify right))
+    )
+    (property "Footprint" "Jumper:SolderJumper-2_P1.3mm_Open_RoundedPad1.0x1.5mm" (at 38.1 74.93 0)
+      (effects (font (size 1.27 1.27)) hide)
+    )
+    (property "Datasheet" "~" (at 38.1 74.93 0)
+      (effects (font (size 1.27 1.27)) hide)
+    )
+    (pin "1")
+    (pin "2")
+    (instances
+      (project "CAN_DISPLAY"
+        (path "/7b7bcc60-3b35-483b-8f75-db7ec854d7bb/0efeef53-f612-43e6-99d4-b53087b36e31"
+          (reference "JP19") (unit 1)
+        )
+        (path "/7b7bcc60-3b35-483b-8f75-db7ec854d7bb/64058649-9106-47b8-8357-4a2d690c60fd"
+          (reference "JP25") (unit 1)
+        )
+      )
+    )
+  )
   (symbol (lib_id "power:GND") (at 143.51 177.8 0) (unit 1)
     (in_bom yes) (on_board yes) (dnp no)
@@
         )
       )
-    )
-  )
-  (symbol (lib_id "Connector:Screw_Terminal_01x04") (at 26.67 82.55 180) (unit 1)
-    (in_bom yes) (on_board yes) (dnp no) (fields_autoplaced)
-    (property "Reference" "J15" (at 26.67 71.12 0)
-      (effects (font (size 1.27 1.27)))
-    )
-    (property "Value" "CHARGER" (at 26.67 73.66 0)
-      (effects (font (size 1.27 1.27)))
-    )
-    (property "Footprint" "TerminalBlock:TerminalBlock_bornier-4_P5.08mm" (at 26.67 82.55 0)
-      (effects (font (size 1.27 1.27)) hide)
-    )
-    (property "Datasheet" "~" (at 26.67 82.55 0)
-      (effects (font (size 1.27 1.27)) hide)
-    )
-    (pin "1")
-    (pin "2")
-    (pin "3")
-    (pin "4")
-    (instances
-      (project "CAN_DISPLAY"
-        (path "/7b7bcc60-3b35-483b-8f75-db7ec854d7bb/6d7ffea3-f61a-415e-92f6-30433f60c362"
-          (reference "J15") (unit 1)
-        )
-        (path "/7b7bcc60-3b35-483b-8f75-db7ec854d7bb/64058649-9106-47b8-8357-4a2d690c60fd"
-          (reference "J17") (unit 1)
-        )
-      )
