File: CAN_DISPLAY/ESP32_sch.kicad_sch (KiCad schematic)
At the start: 37 parts, among them J10 Prodrammer, J11 Micro_SD_Card, J12 J-Link, J15 LED Display, SW1 BOOT, SW2 RESET, U1 ESP32-DevKit, U2 ESP32-WROOM-E

Commit message: PCB Fixes
Parts:
- added J18: J-Link, Connector_PinHeader_2.54mm:PinHeader_2x10_P2.54mm_Vertical, symbol Connector_Generic:Conn_02x10_Odd_Even
- added JP21: JVDD, Jumper:SolderJumper-2_P1.3mm_Open_RoundedPad1.0x1.5mm, symbol Jumper:SolderJumper_2_Open
Connections:
- net +3V3: now also JP21.1 (A)
- net EN: now also J18.15 (Pin_15)
- net GND: now also J18.10 (Pin_10), J18.12 (Pin_12), J18.14 (Pin_14), J18.6 (Pin_6), J18.8 (Pin_8)
- net GPIO_12: now also J18.5 (Pin_5)
- net GPIO_13: now also J18.9 (Pin_9)
- net GPIO_14: now also J18.7 (Pin_7)
- net GPIO_15: now also J18.13 (Pin_13)
- new net: J18.1 (Pin_1), JP21.2 (B)
- no-connect marks 6 -> 15
Other:
- moved on the sheet: J10, J12

Commit message: Add SW
Parts:
- added JP1: BUZZER, Jumper:SolderJumper-2_P1.3mm_Bridged_Pad1.0x1.5mm, symbol Jumper:SolderJumper_2_Bridged
- D4: footprint LED_SMD:LED_1210_3225Metric -> LED_SMD:LED_0805_2012Metric_Pad1.15x1.40mm_HandSolder
- JP1: now left out of the parts list
Connections:
- net GPIO_33_32K: now also JP1.1 (A)
- new net BUZZER: JP1.2 (B)
Other:
- moved on the sheet: JP1

Commit message: Release Version 1.00 Rev 1.00
Connections:
- net GPIO_14: now also JP1.1 (A)
- net GPIO_33_32K: no longer JP1.1 (A)
Changed lines of the file:
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@@
     (fill (type none))
   )
+  (rectangle (start 133.35 160.02) (end 173.99 198.12)
+    (stroke (width 0) (type dash) (color 255 0 2 1))
+    (fill (type none))
+  )
   (rectangle (start 98.425 107.315) (end 161.29 153.035)
     (stroke (width 0) (type default))
@@
     (effects (font (size 1.27 1.27)) (justify right bottom))
   )
-  (label "GPIO_33_32K" (at 69.85 157.48 180) (fields_autoplaced)
-    (effects (font (size 1.27 1.27)) (justify right bottom))
-  )
   (label "GPIO_27" (at 161.29 59.69 180) (fields_autoplaced)
     (effects (font (size 1.27 1.27)) (justify right bottom))
@@
     (effects (font (size 1.27 1.27)) (justify right bottom))
   )
+  (label "GPIO_14" (at 69.85 157.48 180) (fields_autoplaced)
+    (effects (font (size 1.27 1.27)) (justify right bottom))
+  )
