File: LED Matrix Display/ESP32.kicad_sch (KiCad schematic)
At the start: 43 parts, among them J1 I2C Sensor 1, J2 Prodrammer, J3 LED Display, J5 Charger, SW1 BOOT, SW2 RESET, SW3 SW_Reed, U1 ESP32-WROOM-E, U2 BME280, U3 LM2596S-5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

Commit message: LED MX Release candidate
Parts:
- removed C6, C7: 220uF 50V, Capacitor_SMD:CP_Elec_5x5.8, symbol Device:C_Polarized_Small
- removed D6: 12V, LED_SMD:LED_0805_2012Metric_Pad1.15x1.40mm_HandSolder, symbol Device:LED_Small
- removed J3: LED Display, Connector_Molex:Molex_Micro-Fit_3.0_43650-0410_1x04-1MP_P3.00mm_Horizontal_PnP, symbol Connector:Screw_Terminal_01x04
- removed J5: Charger, Connector_Molex:Molex_Micro-Fit_3.0_43650-0410_1x04-1MP_P3.00mm_Horizontal_PnP, symbol Connector:Screw_Terminal_01x04
- removed JP1: Address 0x76 (or 0x77), Jumper:SolderJumper-3_P1.3mm_Bridged12_Pad1.0x1.5mm, symbol Jumper:SolderJumper_3_Bridged12
- removed JP3: 0V, 1Display:NOSILK SolderJumper-2_P1.3mm_Open_Pad1.0x1.5mm, symbol Jumper:SolderJumper_2_Bridged
- removed JP4: SDA, Jumper:SolderJumper-2_P1.3mm_Bridged_Pad1.0x1.5mm, symbol Jumper:SolderJumper_2_Bridged
- removed JP5: SCK, Jumper:SolderJumper-2_P1.3mm_Bridged_Pad1.0x1.5mm, symbol Jumper:SolderJumper_2_Bridged
- removed JP9: SW, Jumper:SolderJumper-2_P1.3mm_Open_RoundedPad1.0x1.5mm, symbol Jumper:SolderJumper_2_Open
- removed L1: 33uH, Inductor_SMD:L_12x12mm_H4.5mm, symbol Device:L_Small
- removed R7: 1K, Resistor_SMD:R_0805_2012Metric_Pad1.20x1.40mm_HandSolder, symbol Device:R_Small
- removed U3: LM2596S-5, Package_TO_SOT_SMD:TO-263-5_TabPin3, symbol Regulator_Switching:LM2596S-5
- added C6: 0.1u, Capacitor_SMD:C_0805_2012Metric_Pad1.18x1.45mm_HandSolder, symbol Device:C_Small
- added D2: BAT54S, Package_TO_SOT_SMD:SOT-23, symbol Diode:BAT54S
- R4: value 4.7K -> 100K
- R5: value 4.7K -> 27K
Connections:
- net GPIO_21 is gone; now on net I2C_SDA: R2.1, U1.33 (GPIO21)
- net GPIO_22 is gone; now on net I2C_SCL: R3.1, U1.36 (GPIO22)
- net +12V: now also R4.2
- net +3V3: now also U2.5 (SDO)
- net +5V: now also D2.2 (K); no longer R4.1
- net GND: now also R5.1, C6.2, D2.1 (A); no longer R5.2
- net GPIO_35: now also R4.1, R5.2, C6.1, D2.3 (COM)
- net GPIO_32_32K renamed ONE_WIRE_2
- net GPIO_33_32K renamed ONE_WIRE
Other:
- note removed: "OPTION LM2596S-ADJ"
- moved on the sheet: C10, C11, C12, C13, C15, C16, C3, C9, U2, U4
