File: LED Matrix Display/LEDS Only.kicad_sch (KiCad schematic)
At the start: 5 parts, among them J5 IN, J5 MINI560, J5 OUT

Commit message: LED MX Release candidate
Parts:
- J5: footprint Connector_Molex:Molex_Micro-Fit_3.0_43650-0410_1x04-1MP_P3.00mm_Horizontal_PnP -> Connector_Molex:Molex_Micro-Fit_3.0_43650-0415_1x04_P3.00mm_Vertical
Connections:
- net ONE_WIRE_2: now reaches J5.2 (Pin_2)
- net ONE_WIRE_2: now also J5.2 (Pin_2)
- net ONE_WIRE: now reaches D1.2 (DOUT), D1.4 (DIN), J5.3 (Pin_3), J5.3 (Pin_3)
- net +12V: now reaches J5.2 (Pin_2), J5.4 (Pin_4), J5.4 (Pin_4)
Other:
- moved on the sheet: J5
Changed lines of the file:
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@@
 (kicad_sch (version 20230121) (generator eeschema)
   (paper "A4")
-  (junction (at 128.27 26.035) (diameter 0) (color 0 0 0 0)
-  )
-  (junction (at 107.95 34.29) (diameter 0) (color 0 0 0 0)
+  (junction (at 86.36 46.99) (diameter 0) (color 0 0 0 0)
+  )
+  (junction (at 77.47 76.2) (diameter 0) (color 0 0 0 0)
   )
   (junction (at 72.39 70.485) (diameter 0) (color 0 0 0 0)
@@
   (junction (at 90.17 73.025) (diameter 0) (color 0 0 0 0)
   )
+  (junction (at 72.39 69.85) (diameter 0) (color 0 0 0 0)
+  )
+  (junction (at 101.6 34.29) (diameter 0) (color 0 0 0 0)
+  )
   (junction (at 80.01 73.025) (diameter 0) (color 0 0 0 0)
   )
-  (wire (pts (xy 80.01 73.025) (xy 80.01 73.66))
+  (junction (at 128.27 25.4) (diameter 0) (color 0 0 0 0)
+  )
+  (wire (pts (xy 80.01 73.025) (xy 80.01 77.47))
     (stroke (width 0) (type default))
   )
@@
     (stroke (width 0) (type default))
   )
-  (wire (pts (xy 86.36 34.29) (xy 107.95 34.29))
+  (wire (pts (xy 86.36 34.29) (xy 101.6 34.29))
+    (stroke (width 0) (type default))
+  )
+  (wire (pts (xy 60.96 76.2) (xy 77.47 76.2))
+    (stroke (width 0) (type default))
+  )
+  (wire (pts (xy 72.39 69.85) (xy 72.39 70.485))
     (stroke (width 0) (type default))
   )
@@
     (stroke (width 0) (type default))
   )
+  (wire (pts (xy 83.82 46.99) (xy 86.36 46.99))
+    (stroke (width 0) (type default))
+  )
   (wire (pts (xy 74.93 72.39) (xy 64.77 72.39))
     (stroke (width 0) (type default))
@@
     (stroke (width 0) (type default))
   )
-  (wire (pts (xy 72.39 66.675) (xy 72.39 70.485))
+  (wire (pts (xy 72.39 66.675) (xy 72.39 69.85))
     (stroke (width 0) (type default))
   )
@@
     (stroke (width 0) (type default))
   )
+  (wire (pts (xy 58.42 69.85) (xy 72.39 69.85))
+    (stroke (width 0) (type default))
+  )
+  (wire (pts (xy 77.47 76.2) (xy 77.47 77.47))
+    (stroke (width 0) (type default))
+  )
   (wire (pts (xy 116.84 24.765) (xy 116.84 26.67))
     (stroke (width 0) (type default))
@@
     (stroke (width 0) (type default))
   )
-  (wire (pts (xy 107.95 26.035) (xy 128.27 26.035))
+  (wire (pts (xy 101.6 25.4) (xy 128.27 25.4))
     (stroke (width 0) (type default))
   )
@@
     (stroke (width 0) (type default))
   )
-  (wire (pts (xy 86.36 68.58) (xy 86.36 34.29))
-    (stroke (width 0) (type default))
-  )
-  (wire (pts (xy 128.27 17.145) (xy 128.27 26.035))
+  (wire (pts (xy 86.36 68.58) (xy 86.36 46.99))
+    (stroke (width 0) (type default))
+  )
+  (wire (pts (xy 128.27 17.145) (xy 128.27 25.4))
     (stroke (width 0) (type default))
   )
@@
     (stroke (width 0) (type default))
   )
-  (wire (pts (xy 107.95 34.29) (xy 109.22 34.29))
-    (stroke (width 0) (type default))
-  )
-  (wire (pts (xy 72.39 70.485) (xy 72.39 73.66))
-    (stroke (width 0) (type default))
-  )
-  (wire (pts (xy 74.93 73.66) (xy 74.93 72.39))
+  (wire (pts (xy 86.36 46.99) (xy 86.36 34.29))
+    (stroke (width 0) (type default))
+  )
+  (wire (pts (xy 101.6 34.29) (xy 109.22 34.29))
+    (stroke (width 0) (type default))
+  )
+  (wire (pts (xy 72.39 70.485) (xy 72.39 77.47))
+    (stroke (width 0) (type default))
+  )
+  (wire (pts (xy 58.42 68.58) (xy 58.42 69.85))
+    (stroke (width 0) (type default))
+  )
+  (wire (pts (xy 74.93 77.47) (xy 74.93 72.39))
     (stroke (width 0) (type default))
   )
@@
     (stroke (width 0) (type default))
   )
+  (wire (pts (xy 77.47 66.675) (xy 77.47 76.2))
+    (stroke (width 0) (type default))
+  )
   (wire (pts (xy 50.8 36.195) (xy 50.8 38.1))
     (stroke (width 0) (type default))
   )
-  (wire (pts (xy 107.95 26.035) (xy 107.95 34.29))
+  (wire (pts (xy 101.6 25.4) (xy 101.6 34.29))
     (stroke (width 0) (type default))
   )
@@
     (stroke (width 0) (type default))
   )
-  (wire (pts (xy 128.27 26.035) (xy 128.27 34.29))
-    (stroke (width 0) (type default))
-  )
   (wire (pts (xy 74.93 66.675) (xy 74.93 68.58))
     (stroke (width 0) (type default))
   )
+  (wire (pts (xy 128.27 25.4) (xy 128.27 34.29))
+    (stroke (width 0) (type default))
+  )
   (wire (pts (xy 80.01 73.025) (xy 90.17 73.025))
     (stroke (width 0) (type default))
+  )
+  (label "ONE_WIRE" (at 118.1675 17.145 0) (fields_autoplaced)
+    (effects (font (size 1.27 1.27)) (justify left bottom))
+  )
+  (label "ONE_WIRE" (at 90.17 34.29 0) (fields_autoplaced)
+    (effects (font (size 1.27 1.27)) (justify left bottom))
+  )
+  (global_label "ONE_WIRE_2" (shape input) (at 60.96 76.2 180) (fields_autoplaced)
+    (effects (font (size 1.27 1.27)) (justify right))
+    (property "Intersheetrefs" "${INTERSHEET_REFS}" (at 46.5449 76.2 0)
+      (effects (font (size 1.27 1.27)) (justify right) hide)
+    )
+  )
+  (global_label "ONE_WIRE" (shape input) (at 83.82 46.99 180) (fields_autoplaced)
+    (effects (font (size 1.27 1.27)) (justify right))
+    (property "Intersheetrefs" "${INTERSHEET_REFS}" (at 71.582 46.99 0)
+      (effects (font (size 1.27 1.27)) (justify right) hide)
+    )
   )
   (symbol (lib_id "power:GND") (at 50.8 45.72 0) (unit 1)
@@
     )
   )
-  (symbol (lib_id "Connector:Screw_Terminal_01x04") (at 77.47 78.74 270) (unit 1)
+  (symbol (lib_id "Connector:Screw_Terminal_01x04") (at 77.47 82.55 270) (unit 1)
     (in_bom yes) (on_board yes) (dnp no)
-    (property "Reference" "J5" (at 76.2 85.09 90)
-      (effects (font (size 1.27 1.27)))
-    )
-    (property "Value" "OUT" (at 76.2 82.55 90)
-      (effects (font (size 1.27 1.27)))
-    )
-    (property "Footprint" "Connector_Molex:Molex_Micro-Fit_3.0_43650-0410_1x04-1MP_P3.00mm_Horizontal_PnP" (at 77.47 78.74 0)
-      (effects (font (size 1.27 1.27)) hide)
-    )
-    (property "Datasheet" "~" (at 77.47 78.74 0)
+    (property "Reference" "J5" (at 76.2 88.9 90)
+      (effects (font (size 1.27 1.27)))
+    )
+    (property "Value" "OUT" (at 76.2 86.36 90)
+      (effects (font (size 1.27 1.27)))
+    )
+    (property "Footprint" "Connector_Molex:Molex_Micro-Fit_3.0_43650-0415_1x04_P3.00mm_Vertical" (at 77.47 82.55 0)
+      (effects (font (size 1.27 1.27)) hide)
+    )
+    (property "Datasheet" "~" (at 77.47 82.55 0)
       (effects (font (size 1.27 1.27)) hide)
     )
@@
     )
   )
+  (symbol (lib_id "power:+12V") (at 58.42 68.58 0) (unit 1)
+    (in_bom yes) (on_board yes) (dnp no) (fields_autoplaced)
+    (property "Reference" "#PWR014" (at 58.42 72.39 0)
+      (effects (font (size 1.27 1.27)) hide)
+    )
+    (property "Value" "+12V" (at 58.42 63.5 0)
+      (effects (font (size 1.27 1.27)))
+    )
+    (property "Footprint" "" (at 58.42 68.58 0)
+      (effects (font (size 1.27 1.27)) hide)
+    )
+    (property "Datasheet" "" (at 58.42 68.58 0)
+      (effects (font (size 1.27 1.27)) hide)
+    )
+    (pin "1")
+    (instances
+      (project "LED Matrix Display"
+        (path "/02d83b85-cfa3-4125-bdd4-4666ac4bec4b/3ffbcd43-3a32-410d-bdaf-78046e2ef2b3"
+          (reference "#PWR014") (unit 1)
+        )
+        (path "/02d83b85-cfa3-4125-bdd4-4666ac4bec4b/a5c4692e-8268-4e5f-99a8-3858d34e691b"
+          (reference "#PWR030") (unit 1)
+        )
+      )
+      (project "CAN_DISPLAY"
+        (path "/7b7bcc60-3b35-483b-8f75-db7ec854d7bb/64058649-9106-47b8-8357-4a2d690c60fd"
+          (reference "#PWR070") (unit 1)
+        )
+      )
+    )
+  )
   (symbol (lib_id "Connector:Screw_Terminal_01x04") (at 77.47 61.595 270) (mirror x) (unit 1)
     (in_bom yes) (on_board yes) (dnp no)
@@
       (effects (font (size 1.27 1.27)))
     )
-    (property "Footprint" "Connector_Molex:Molex_Micro-Fit_3.0_43650-0410_1x04-1MP_P3.00mm_Horizontal_PnP" (at 77.47 61.595 0)
-      (effects (font (size 1.27 1.27)) hide)
-    )
+    (property "Footprint" "Connector_Molex:Molex_Micro-Fit_3.0_43650-0415_1x04_P3.00mm_Vertical" (at 77.47 61.595 0)
+      (effects (font (size 1.27 1.27)) hide)
+    )
